File: awatch2.sch (KiCad schematic (older format))
At the start: 17 parts, among them J101 Conn_01x02, J102 Conn_01x02, J103 Conn_01x02, J104 Conn_01x02, SW101 B3S-1000, SW102 B3S-1000, SW103 B3S-1000, SW104 B3S-1000

Commit message: PMIC relative placement and routing
Parts:
- J102, J103: footprint Connector_PinSocket_2.54mm:PinSocket_1x02_P2.54mm_Vertical -> Connector_PinHeader_2.54mm:PinHeader_1x02_P2.54mm_Vertical
Changed lines of the file:
@@
 F 0 "J102" H 2520 2625 50  0000 C CNN
 F 1 "Conn_01x02" H 2520 2716 50  0000 C CNN
-F 2 "Connector_PinSocket_2.54mm:PinSocket_1x02_P2.54mm_Vertical" H 2600 2950 50  0001 C CNN
+F 2 "Connector_PinHeader_2.54mm:PinHeader_1x02_P2.54mm_Vertical" H 2600 2950 50  0001 C CNN
 F 3 "~" H 2600 2950 50  0001 C CNN
 	1    2600 2950
@@
 F 0 "J103" H 2520 3075 50  0000 C CNN
 F 1 "Conn_01x02" H 2520 3166 50  0000 C CNN
-F 2 "Connector_PinSocket_2.54mm:PinSocket_1x02_P2.54mm_Vertical" H 2600 3400 50  0001 C CNN
+F 2 "Connector_PinHeader_2.54mm:PinHeader_1x02_P2.54mm_Vertical" H 2600 3400 50  0001 C CNN
 F 3 "~" H 2600 3400 50  0001 C CNN
 	1    2600 3400

Commit message: approx. final layout
Parts:
- J101, J104: footprint Connector_PinSocket_2.54mm:PinSocket_1x02_P2.54mm_Vertical -> Connector_PinHeader_2.54mm:PinHeader_1x02_P2.54mm_Vertical
- SW101, SW102, SW103, SW104: DigiKey PN (none) -> SW836CT-ND
Changed lines of the file:
@@
 $Descr A4 11693 8268
 encoding utf-8
-Sheet 1 9
+Sheet 1 10
 Title "AWatch2"
 Date ""
@@
 F 0 "J104" H 3520 2325 50  0000 C CNN
 F 1 "Conn_01x02" H 3520 2416 50  0000 C CNN
-F 2 "Connector_PinSocket_2.54mm:PinSocket_1x02_P2.54mm_Vertical" H 3600 2650 50  0001 C CNN
+F 2 "Connector_PinHeader_2.54mm:PinHeader_1x02_P2.54mm_Vertical" H 3600 2650 50  0001 C CNN
 F 3 "~" H 3600 2650 50  0001 C CNN
 	1    3600 2650
@@
 F 2 "Button_Switch_SMD:SW_SPST_B3S-1000" H 4350 5600 50  0001 C CNN
 F 3 "" H 4350 5600 50  0001 C CNN
+F 4 "SW836CT-ND" H 0   0   50  0001 C CNN "DigiKey PN"
 	1    4350 5400
 	0    -1   -1   0
@@
 F 2 "Button_Switch_SMD:SW_SPST_B3S-1000" H 4450 5600 50  0001 C CNN
 F 3 "" H 4450 5600 50  0001 C CNN
+F 4 "SW836CT-ND" H 0   0   50  0001 C CNN "DigiKey PN"
 	1    4450 5400
 	0    -1   -1   0
@@
 F 2 "Button_Switch_SMD:SW_SPST_B3S-1000" H 4550 5600 50  0001 C CNN
 F 3 "" H 4550 5600 50  0001 C CNN
+F 4 "SW836CT-ND" H 0   0   50  0001 C CNN "DigiKey PN"
 	1    4550 5400
 	0    -1   -1   0
@@
 F 2 "Button_Switch_SMD:SW_SPST_B3S-1000" H 4650 5600 50  0001 C CNN
 F 3 "" H 4650 5600 50  0001 C CNN
+F 4 "SW836CT-ND" H 0   0   50  0001 C CNN "DigiKey PN"
 	1    4650 5400
 	0    -1   -1   0
@@
 F 0 "J101" H 2420 4075 50  0000 C CNN
 F 1 "Conn_01x02" H 2420 4166 50  0000 C CNN
-F 2 "Connector_PinSocket_2.54mm:PinSocket_1x02_P2.54mm_Vertical" H 2500 4400 50  0001 C CNN
+F 2 "Connector_PinHeader_2.54mm:PinHeader_1x02_P2.54mm_Vertical" H 2500 4400 50  0001 C CNN
 F 3 "~" H 2500 4400 50  0001 C CNN
 	1    2500 4400
@@
 Wire Wire Line
 	6900 3450 6650 3450
+$Sheet
+S 9200 1800 850  500
+U 5C43713C
+F0 "Mounting holes" 50
+F1 "awatch-mounting.sch" 50
+$EndSheet
 $EndSCHEMATC

Commit message: BOM fully populated
Parts:
- J101, J102, J103, J104: DigiKey PN (none) -> S1011EC-02-ND, S9341-ND
Changed lines of the file:
@@
 F 2 "Connector_PinHeader_2.54mm:PinHeader_1x02_P2.54mm_Vertical" H 3600 2650 50  0001 C CNN
 F 3 "~" H 3600 2650 50  0001 C CNN
+F 4 "S1011EC-02-ND, S9341-ND" H 0   0   50  0001 C CNN "DigiKey PN"
 	1    3600 2650
 	-1   0    0    1
@@
 F 2 "Connector_PinHeader_2.54mm:PinHeader_1x02_P2.54mm_Vertical" H 2600 2950 50  0001 C CNN
 F 3 "~" H 2600 2950 50  0001 C CNN
+F 4 "S1011EC-02-ND, S9341-ND" H 0   0   50  0001 C CNN "DigiKey PN"
 	1    2600 2950
 	-1   0    0    1
@@
 F 2 "Connector_PinHeader_2.54mm:PinHeader_1x02_P2.54mm_Vertical" H 2600 3400 50  0001 C CNN
 F 3 "~" H 2600 3400 50  0001 C CNN
+F 4 "S1011EC-02-ND, S9341-ND" H 0   0   50  0001 C CNN "DigiKey PN"
 	1    2600 3400
 	-1   0    0    1
@@
 F 2 "Connector_PinHeader_2.54mm:PinHeader_1x02_P2.54mm_Vertical" H 2500 4400 50  0001 C CNN
 F 3 "~" H 2500 4400 50  0001 C CNN
+F 4 "S1011EC-02-ND, S9341-ND" H 0   0   50  0001 C CNN "DigiKey PN"
 	1    2500 4400
 	-1   0    0    1
